File: Sparkdog PF-DI V3/Knock.sch (KiCad schematic (older format))
At the start: 23 parts, among them U400 TLV9052, U401 TLV9052

Commit message: Running changes backup
Parts:
- U400, U401: footprint Samacsys:SOT65P280X110-8N -> Samacsys:SOP65P640X120-8N
Changed lines of the file:
@@
 F 0 "U400" H 5100 2117 50  0000 C CNN
 F 1 "TLV9052" H 5100 2026 50  0000 C CNN
-F 2 "Samacsys:SOT65P280X110-8N" H 5100 1750 50  0001 C CNN
+F 2 "Samacsys:SOP65P640X120-8N" H 5100 1750 50  0001 C CNN
 F 3 "https://www.analog.com/media/en/technical-documentation/data-sheets/AD8610_8620.pdf" H 5100 1750 50  0001 C CNN
 	1    5100 1750
@@
 F 0 "U400" H 5250 2867 50  0000 C CNN
 F 1 "TLV9052" H 5250 2776 50  0000 C CNN
-F 2 "Samacsys:SOT65P280X110-8N" H 5250 2500 50  0001 C CNN
+F 2 "Samacsys:SOP65P640X120-8N" H 5250 2500 50  0001 C CNN
 F 3 "https://www.analog.com/media/en/technical-documentation/data-sheets/AD8610_8620.pdf" H 5250 2500 50  0001 C CNN
 	2    5250 2500
@@
 F 0 "U400" H 6308 2096 50  0000 L CNN
 F 1 "TLV9052" H 6308 2005 50  0000 L CNN
-F 2 "Samacsys:SOT65P280X110-8N" H 6350 2050 50  0001 C CNN
+F 2 "Samacsys:SOP65P640X120-8N" H 6350 2050 50  0001 C CNN
 F 3 "https://www.analog.com/media/en/technical-documentation/data-sheets/AD8610_8620.pdf" H 6350 2050 50  0001 C CNN
 	3    6350 2050
@@
 F 0 "U401" H 5400 4267 50  0000 C CNN
 F 1 "TLV9052" H 5400 4176 50  0000 C CNN
-F 2 "Samacsys:SOT65P280X110-8N" H 5400 3900 50  0001 C CNN
+F 2 "Samacsys:SOP65P640X120-8N" H 5400 3900 50  0001 C CNN
 F 3 "https://www.analog.com/media/en/technical-documentation/data-sheets/AD8610_8620.pdf" H 5400 3900 50  0001 C CNN
 	1    5400 3900
@@
 F 0 "U401" H 5400 5117 50  0000 C CNN
 F 1 "TLV9052" H 5400 5026 50  0000 C CNN
-F 2 "Samacsys:SOT65P280X110-8N" H 5400 4750 50  0001 C CNN
+F 2 "Samacsys:SOP65P640X120-8N" H 5400 4750 50  0001 C CNN
 F 3 "https://www.analog.com/media/en/technical-documentation/data-sheets/AD8610_8620.pdf" H 5400 4750 50  0001 C CNN
 	2    5400 4750
@@
 F 0 "U401" H 6308 4246 50  0000 L CNN
 F 1 "TLV9052" H 6308 4155 50  0000 L CNN
-F 2 "Samacsys:SOT65P280X110-8N" H 6350 4200 50  0001 C CNN
+F 2 "Samacsys:SOP65P640X120-8N" H 6350 4200 50  0001 C CNN
 F 3 "https://www.analog.com/media/en/technical-documentation/data-sheets/AD8610_8620.pdf" H 6350 4200 50  0001 C CNN
 	3    6350 4200
