File: Sparkdog PF-DI V3/Sparkdog PF-DI V3.sch (KiCad schematic (older format))
At the start: 9 parts, among them J1 Conn_01x06_Female, J2 Conn_01x08_Female, J3 Conn_01x06_Female, J4 Conn_01x08_Female, J5 Conn_01x06_Female, J6 Conn_01x08_Female, U2 Arduino_Footprint

Commit message: Running changes backup
Parts:
- added RN100, RN101: 1206 1k, Samacsys:742C083103JP, symbol Device:R_Pack04
Connections:
- net labels added: BM_RX, BM_TX, IO_PWM7
- net labels removed: UART_RX, UART_TX
- wire segments 224 -> 231
Other:
- moved on the sheet: J6
Changed lines of the file:
@@
 F18 "SIGA_LV_EN" O R 4400 7850 50
 F19 "SIGB_LV_EN" O R 4400 7950 50
-F20 "SIG_PUMP_PWM" I L 3100 8950 50
+F20 "SIG_PUMP_PWM" I L 3100 8855 50
 F21 "SIG_PUMP_PWMS" O R 4400 8750 50
 $EndSheet
@@
 Wire Wire Line
 	4400 8650 4650 8650
-$Sheet
-S 10300 6750 950  1675
-U 60C1F65F
-F0 "5 ETC" 50
-F1 "ETC.sch" 50
-F2 "ETC_ENA" I L 10300 6850 50
-F3 "ETC_ENB" I L 10300 6950 50
-F4 "ETC_IN1A" I L 10300 7050 50
-F5 "ETC_IN1B" I L 10300 7150 50
-F6 "ETC_IN2A" I L 10300 7250 50
-F7 "ETC_IN2B" I L 10300 7350 50
-F8 "ETC_O2A" O R 11250 6850 50
-F9 "ETC_O2B" O R 11250 6950 50
-F10 "ETC_O1A" O R 11250 7050 50
-F11 "ETC_O1B" O R 11250 7150 50
-F12 "ETC_VFF" I L 10300 7450 50
-F13 "ETC_VFB" I L 10300 7550 50
-F14 "ETC_IFA" O R 11250 7450 50
-F15 "ETC_IFB" O R 11250 7550 50
-F16 "SCLK" I R 11250 7250 50
-F17 "MOSI" I R 11250 7350 50
-F18 "IO_PWM1" O R 11250 7650 50
-F19 "IO_PWM2" O R 11250 7750 50
-F20 "IO_PWM3" O R 11250 7850 50
-F21 "IO_PWM4" O R 11250 7950 50
-F22 "IO_PWM5" O R 11250 8050 50
-F23 "IO_PWM6" O R 11250 8150 50
-F24 "IO_PWM7" O R 11250 8250 50
-F25 "IO_PWM8" O R 11250 8350 50
-$EndSheet
 Wire Wire Line
 	9300 8600 9650 8600
@@
 $EndComp
 Wire Wire Line
-	2750 5600 2400 5600
-Wire Wire Line
-	2400 5700 2750 5700
-Wire Wire Line
-	2400 5500 2750 5500
+	2275 5600 1925 5600
+Wire Wire Line
+	1925 5700 2275 5700
+Wire Wire Line
+	1925 5500 2275 5500
 Wire Wire Line
 	4650 9050 4400 9050
@@
 Wire Wire Line
 	6300 9000 6900 9000
-Text Label 3050 8950 2    50   ~ 0
+Text Label 3090 8855 2    50   ~ 0
 SIG_GDIP_EN
-Wire Wire Line
-	3100 8950 2550 8950
 Text Label 8050 9500 0    50   ~ 0
 SIGAB_HVEN
@@
 	9300 8350 9750 8350
 Text Label 9400 8250 0    50   ~ 0
-UART_TX
+BM_TX
 Text Label 9400 8350 0    50   ~ 0
-UART_RX
+BM_RX
 Wire Wire Line
 	6300 5550 6300 6100
@@
 	5300 3250 5050 3250
 Wire Wire Line
-	2400 5400 2750 5400
-Wire Wire Line
-	2750 5300 2400 5300
-Wire Wire Line
-	2750 5200 2400 5200
-Text Label 2625 5200 0    50   ~ 0
+	1925 5400 2275 5400
+Wire Wire Line
+	2275 5300 1925 5300
+Wire Wire Line
+	2275 5200 1925 5200
+Text Label 2050 5200 0    50   ~ 0
 T1
-Text Label 2625 5300 0    50   ~ 0
+Text Label 2050 5300 0    50   ~ 0
 T2
-Text Label 2625 5400 0    50   ~ 0
+Text Label 2050 5400 0    50   ~ 0
 T3
-Text Label 2625 5500 0    50   ~ 0
+Text Label 2050 5500 0    50   ~ 0
 T4
-Text Label 2625 5600 0    50   ~ 0
+Text Label 2050 5600 0    50   ~ 0
 T5
-Text Label 2625 5700 0    50   ~ 0
+Text Label 2050 5700 0    50   ~ 0
 T6
 $Comp
 L Connector:Conn_01x08_Female J6
 U 1 1 662BA502
-P 12250 7950
-F 0 "J6" H 12278 7926 50  0000 L CNN
-F 1 "Conn_01x08_Female" H 11800 8350 50  0000 L CNN
-F 2 "Sparkdog PF-DI V3:SIP-8" H 12250 7950 50  0001 C CNN
-F 3 "~" H 12250 7950 50  0001 C CNN
-	1    12250 7950
+P 12245 7750
+F 0 "J6" H 12273 7726 50  0000 L CNN
+F 1 "Conn_01x08_Female" H 11795 8150 50  0000 L CNN
+F 2 "Sparkdog PF-DI V3:SIP-8" H 12245 7750 50  0001 C CNN
+F 3 "~" H 12245 7750 50  0001 C CNN
+	1    12245 7750
 	1    0    0    -1
 $EndComp
 Wire Wire Line
-	12050 8250 11250 8250
-Wire Wire Line
-	11250 8350 12050 8350
-Wire Wire Line
-	11250 8150 12050 8150
-Wire Wire Line
-	11250 8050 12050 8050
-Wire Wire Line
-	12050 7950 11250 7950
-Wire Wire Line
-	12050 7850 11250 7850
-Wire Wire Line
-	11250 7750 12050 7750
-Wire Wire Line
-	11250 7650 12050 7650
-Wire Bus Line
-	10700 2825 10700 3625
-Wire Bus Line
-	6150 6200 8100 6200
-Wire Bus Line
-	13625 3325 13625 6200
-Wire Bus Line
-	8100 6200 8100 7450
-Wire Bus Line
-	4600 3650 4600 4900
-Wire Bus Line
-	7975 7600 7975 8800
+	11830 8250 11250 8250
+Wire Wire Line
+	12045 7950 11250 7950
+Wire Wire Line
+	12045 7850 11250 7850
+Wire Wire Line
+	11250 7750 12045 7750
+Wire Wire Line
+	11250 7650 12045 7650
 Text Label 2800 6200 0    50   ~ 0
 DB1
+$Comp
+L Device:R_Pack04 RN?
+U 1 1 6693AA30
+P 2475 5500
+AR Path="/60717C73/6693AA30" Ref="RN?"  Part="1"
+AR Path="/6693AA30" Ref="RN101"  Part="1"
+F 0 "RN101" V 2000 5550 50  0000 L CNN
+F 1 "1206 1k" V 2000 5175 50  0000 L CNN
+F 2 "Samacsys:742C083103JP" V 2750 5500 50  0001 C CNN
+F 3 "~" H 2475 5500 50  0001 C CNN
+	1    2475 5500
+	0    -1   -1   0
+$EndComp
+$Comp
+L Device:R_Pack04 RN?
+U 1 1 6694E9B5
+P 2475 5100
+AR Path="/60717C73/6694E9B5" Ref="RN?"  Part="1"
+AR Path="/6694E9B5" Ref="RN100"  Part="1"
+F 0 "RN100" V 1700 5150 50  0000 L CNN
+F 1 "1206 1k" V 1700 4775 50  0000 L CNN
+F 2 "Samacsys:742C083103JP" V 2750 5100 50  0001 C CNN
+F 3 "~" H 2475 5100 50  0001 C CNN
+	1    2475 5100
+	0    -1   -1   0
+$EndComp
+Wire Wire Line
+	2675 5000 2750 5000
+Wire Wire Line
+	2675 5100 2750 5100
+Wire Wire Line
+	2675 5200 2750 5200
+Wire Wire Line
+	2675 5300 2750 5300
+Wire Wire Line
+	2675 5400 2750 5400
+Wire Wire Line
+	2675 5500 2750 5500
+Wire Wire Line
+	2675 5600 2750 5600
+Wire Wire Line
+	2675 5700 2750 5700
+$Sheet
+S 10300 6750 950  1675
+U 60C1F65F
+F0 "5 ETC" 50
+F1 "ETC.sch" 50
+F2 "ETC_ENA" I L 10300 6850 50
+F3 "ETC_ENB" I L 10300 6950 50
+F4 "ETC_IN1A" I L 10300 7050 50
+F5 "ETC_IN1B" I L 10300 7150 50
+F6 "ETC_IN2A" I L 10300 7250 50
+F7 "ETC_IN2B" I L 10300 7350 50
+F8 "ETC_O2A" O R 11250 6850 50
+F9 "ETC_O2B" O R 11250 6950 50
+F10 "ETC_O1A" O R 11250 7050 50
+F11 "ETC_O1B" O R 11250 7150 50
+F12 "ETC_VFF" I L 10300 7450 50
+F13 "ETC_VFB" I L 10300 7550 50
+F14 "ETC_IFA" O R 11250 7450 50
+F15 "ETC_IFB" O R 11250 7550 50
+F16 "SCLK" I R 11250 7250 50
+F17 "MOSI" I R 11250 7350 50
+F18 "IO_PWM1" O R 11250 7650 50
+F19 "IO_PWM2" O R 11250 7750 50
+F20 "IO_PWM3" O R 11250 8050 50
+F21 "IO_PWM4" O R 11250 8150 50
+F22 "IO_PWM5" O R 11250 7850 50
+F23 "IO_PWM6" O R 11250 7950 50
+$EndSheet
+Wire Wire Line
+	11250 8050 12045 8050
+Wire Wire Line
+	12045 8150 11250 8150
+Text HLabel 11250 8250 0    50   Output ~ 0
+IO_PWM7
+Text Label 11310 8250 0    50   ~ 0
+SIG_GDIP_EN
+Wire Wire Line
+	3100 8855 2600 8855
+Wire Bus Line
+	10700 2825 10700 3625
+Wire Bus Line
+	6150 6200 8100 6200
+Wire Bus Line
+	13625 3325 13625 6200
+Wire Bus Line
+	8100 6200 8100 7450
+Wire Bus Line
+	4600 3650 4600 4900
+Wire Bus Line
+	7975 7600 7975 8800
 $EndSCHEMATC
